File: PCB/OxFloodNet_sensor.brd (EAGLE design)
At the start: 45 x 57.1 mm, 18 parts, among them CN1 1x3W, IC1 DS1820, Q1 MOSFET-NCHANNEL2N7000, U1 POWER-POD, X1 u.FL

Commit message: Updated to v3.1
Parts:
- moved +VE 0.64 mm to (31.9, 18.4), turned to 270 degrees
- moved U1 0.63 mm to (29.0, 8.37)
- turned -VE to 270 degrees
Routing:
- net 3.3V: track 88.5 -> 95.2 mm
- net N$3: track 6.21 -> 8.13 mm
Changed lines of the file:
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@@
 <element name="ANT1" library="wirepad" package="2,54/0,8" value="Antenna Pad" x="2.54" y="26.67"/>
 <element name="X1" library="adafruit" package="U.FL" value="u.FL" x="3.81" y="19.05" rot="R90"/>
-<element name="-VE" library="wirepad" package="2,54/0,8" value="" x="32.09" y="22.39"/>
-<element name="+VE" library="wirepad" package="2,54/0,8" value="" x="31.91" y="17.81"/>
-<element name="U1" library="Ciseco Footprints" package="POWER-POD-LANDING" value="POWER-POD" x="29" y="9" rot="R270"/>
+<element name="-VE" library="wirepad" package="2,54/0,8" value="" x="32.09" y="22.39" rot="R270"/>
+<element name="+VE" library="wirepad" package="2,54/0,8" value="" x="31.91" y="18.445" rot="R270"/>
+<element name="U1" library="Ciseco Footprints" package="POWER-POD-LANDING" value="POWER-POD" x="29" y="8.365" rot="R270"/>
 <element name="C2" library="rcl" package="C025-024X044" value="100nF" x="4" y="14"/>
 <element name="C1" library="rcl" package="C025-024X044" value="100nF" x="8" y="28"/>
@@
 <wire x1="19.304" y1="21.336" x2="19.52" y2="21.23" width="0.4" layer="16"/>
 <wire x1="5.588" y1="23.368" x2="5.4" y2="23.37" width="0.4" layer="16"/>
-<wire x1="34.036" y1="7.62" x2="33.02" y2="7.62" width="0.4" layer="16"/>
-<wire x1="33.02" y1="7.62" x2="29" y2="7.73" width="0.4" layer="16"/>
-<wire x1="34.036" y1="7.62" x2="34.29" y2="7.67919375" width="0.4" layer="16"/>
 <contactref element="C3" pad="+"/>
 <contactref element="C1" pad="1"/>
@@
 <wire x1="19.812" y1="20.828" x2="19.52" y2="21.23" width="0.4" layer="1"/>
 <wire x1="25.4" y1="19.812" x2="25" y2="20.27" width="0.4" layer="16"/>
-<wire x1="34.036" y1="11.176" x2="34.29" y2="11.176" width="0.4" layer="16"/>
 <wire x1="6.604" y1="24.892" x2="6.604" y2="27.94" width="0.4" layer="1"/>
 <wire x1="5.588" y1="23.876" x2="6.604" y2="24.892" width="0.4" layer="1"/>
@@
 <wire x1="2.8" y1="52.4" x2="2.54" y2="52.07" width="0.4" layer="1"/>
 <wire x1="2.8" y1="54.4" x2="2.54" y2="54.61" width="0.4" layer="1"/>
-<wire x1="34.036" y1="11.176" x2="29.845" y2="15.367" width="0.4064" layer="16"/>
-<wire x1="29.845" y1="15.367" x2="25.4" y2="19.812" width="0.4064" layer="16"/>
 <wire x1="3.048" y1="31.242" x2="3.048" y2="51.816" width="0.4" layer="1"/>
 <wire x1="6.096" y1="28.194" x2="3.048" y2="31.242" width="0.4" layer="1"/>
 <wire x1="3.048" y1="51.816" x2="2.54" y2="52.07" width="0.4" layer="1"/>
 <wire x1="6.096" y1="28.194" x2="6.73" y2="28" width="0.4" layer="1"/>
-<wire x1="28.194" y1="25.908" x2="27.432" y2="25.908" width="0.4" layer="16"/>
-<wire x1="29.718" y1="24.384" x2="28.194" y2="25.908" width="0.4" layer="16"/>
-<wire x1="29.718" y1="15.24" x2="29.718" y2="24.384" width="0.4" layer="16"/>
+<wire x1="34.29" y1="7.62" x2="29.718" y2="7.62" width="0.4" layer="16"/>
+<wire x1="29.718" y1="7.62" x2="29" y2="7.095" width="0.4" layer="16"/>
+<wire x1="31.242" y1="25.908" x2="29.718" y2="25.908" width="0.4" layer="16"/>
+<wire x1="29.718" y1="25.908" x2="27.432" y2="25.908" width="0.4" layer="16"/>
+<wire x1="44.196" y1="12.954" x2="31.242" y2="25.908" width="0.4" layer="16"/>
 <wire x1="27.432" y1="25.908" x2="27.1742" y2="26.4795" width="0.4" layer="16"/>
-<wire x1="29.718" y1="15.24" x2="29.845" y2="15.367" width="0.4" layer="16"/>
+<wire x1="44.196" y1="12.954" x2="44.196" y2="12.699996875" width="0.4" layer="16"/>
+<wire x1="29.718" y1="22.86" x2="29.718" y2="25.908" width="0.4" layer="16"/>
+<wire x1="28.956" y1="22.098" x2="29.718" y2="22.86" width="0.4" layer="16"/>
+<wire x1="26.67" y1="22.098" x2="28.956" y2="22.098" width="0.4" layer="16"/>
+<wire x1="25.146" y1="20.574" x2="26.67" y2="22.098" width="0.4" layer="16"/>
+<wire x1="25.146" y1="20.574" x2="25" y2="20.27" width="0.4" layer="16"/>
 </signal>
 <signal name="N$4">
@@
 <contactref element="U1" pad="1"/>
 <contactref element="+VE" pad="1"/>
-<wire x1="29.2" y1="15.2" x2="29.2" y2="13.2" width="0.4" layer="1"/>
-<wire x1="31.6" y1="17.6" x2="29.2" y2="15.2" width="0.4" layer="1"/>
-<wire x1="29.2" y1="13.2" x2="29" y2="12.81" width="0.4" layer="1"/>
-<wire x1="31.6" y1="17.6" x2="31.91" y2="17.81" width="0.4" layer="1"/>
+<wire x1="29.718" y1="16.764" x2="29.718" y2="12.192" width="0.4" layer="1"/>
+<wire x1="31.242" y1="18.288" x2="29.718" y2="16.764" width="0.4" layer="1"/>
+<wire x1="29.718" y1="12.192" x2="29" y2="12.175" width="0.4" layer="1"/>
+<wire x1="31.242" y1="18.288" x2="31.91" y2="18.445" width="0.4" layer="1"/>
 </signal>
 </signals>
